File: PCB/sampler.sch (KiCad schematic (older format))
At the start: 7 parts, among them J1 CONN_02X15, U1 AD9200JRSZ

Commit message: pcb bugfix.
Parts:
- C1, C2: value 1uF -> 0.1uF
- C3, C4: value C -> 0.1uF
- C5: value C -> 10uF
Connections:
- net analog-ground: now reaches C1.2, C2.2, C4.2, J1.2 (P2), J1.5 (P5), J1.7 (P7), J1.9 (P9), U1.1 (AVSS)
- net analog-ground: now also J1.13 (P13), J1.15 (P15)
- net upper-ref-V: now reaches C3.2, C4.1, C5.2, U1.21 (REFTS), U1.22 (REFTF)
- net upper-ref-V: now also J1.29 (P29)
- net lower-ref-V: now reaches C2.1, C3.1, C5.1, J1.30 (P30), U1.24 (REFBF), U1.25 (REFBS)
- net lower-ref-V: no longer J1.29 (P29)

Commit message: pcb update
Parts:
- C1, C2, C3, C4: footprint (none) -> Capacitors_SMD:C_0805
- C5: footprint (none) -> Capacitors_SMD:C_0603
- J1: footprint (none) -> Socket_Strips:Socket_Strip_Straight_2x15_Pitch2.54mm_SMD
- U1: footprint (none) -> Housings_SSOP:SSOP-28_5.3x10.2mm_Pitch0.65mm
Changed lines of the file:
@@
 LIBS:contrib
 LIBS:valves
+LIBS:sampler-cache
 EELAYER 25 0
 EELAYER END
@@
 F 0 "U1" H 6750 2750 60  0000 C CNN
 F 1 "AD9200JRSZ" H 6750 2750 60  0000 C CNN
-F 2 "" H 6750 2750 60  0001 C CNN
+F 2 "Housings_SSOP:SSOP-28_5.3x10.2mm_Pitch0.65mm" H 6750 2750 60  0001 C CNN
 F 3 "" H 6750 2750 60  0001 C CNN
 	1    6750 2750
@@
 F 0 "J1" H 2300 3250 50  0000 C CNN
 F 1 "CONN_02X15" V 2300 2450 50  0000 C CNN
-F 2 "" H 2300 1300 50  0001 C CNN
+F 2 "Socket_Strips:Socket_Strip_Straight_2x15_Pitch2.54mm_SMD" H 2300 1300 50  0001 C CNN
 F 3 "" H 2300 1300 50  0001 C CNN
 	1    2300 2450
@@
 F 0 "C1" H 10275 1800 50  0000 L CNN
 F 1 "0.1uF" H 10275 1600 50  0000 L CNN
-F 2 "" H 10288 1550 50  0001 C CNN
+F 2 "Capacitors_SMD:C_0805" H 10288 1550 50  0001 C CNN
 F 3 "" H 10250 1700 50  0001 C CNN
 	1    10250 1700
@@
 F 0 "C2" H 10025 2500 50  0000 L CNN
 F 1 "0.1uF" H 10025 2300 50  0000 L CNN
-F 2 "" H 10038 2250 50  0001 C CNN
+F 2 "Capacitors_SMD:C_0805" H 10038 2250 50  0001 C CNN
 F 3 "" H 10000 2400 50  0001 C CNN
 	1    10000 2400
@@
 F 0 "C3" H 10025 3150 50  0000 L CNN
 F 1 "0.1uF" H 10025 2950 50  0000 L CNN
-F 2 "" H 10038 2900 50  0001 C CNN
+F 2 "Capacitors_SMD:C_0805" H 10038 2900 50  0001 C CNN
 F 3 "" H 10000 3050 50  0001 C CNN
 	1    10000 3050
@@
 F 0 "C5" H 10375 3150 50  0000 L CNN
 F 1 "10uF" H 10375 2950 50  0000 L CNN
-F 2 "" H 10388 2900 50  0001 C CNN
+F 2 "Capacitors_SMD:C_0603" H 10388 2900 50  0001 C CNN
 F 3 "" H 10350 3050 50  0001 C CNN
 	1    10350 3050
@@
 F 0 "C4" H 10025 3850 50  0000 L CNN
 F 1 "0.1uF" H 10025 3650 50  0000 L CNN
-F 2 "" H 10038 3600 50  0001 C CNN
+F 2 "Capacitors_SMD:C_0805" H 10038 3600 50  0001 C CNN
 F 3 "" H 10000 3750 50  0001 C CNN
 	1    10000 3750
