File: PCB/sampler.kicad_pcb (KiCad board)
At the start: 2 copper layers, 0 parts

Commit message: pcb update
Parts:
- added C1: 0.1uF, Capacitors_SMD:C_0805, F.Cu at (181.6, 111.8)
- added C2: 0.1uF, Capacitors_SMD:C_0805, F.Cu at (179.1, 96.5)
- added C3: 0.1uF, Capacitors_SMD:C_0805, F.Cu at (172.7, 91.4)
- added C4: 0.1uF, Capacitors_SMD:C_0805, F.Cu at (179.1, 105.4)
- added C5: 10uF, Capacitors_SMD:C_0603, F.Cu at (185.4, 99.1)
- added J1: CONN_02X15, Socket_Strips:Socket_Strip_Straight_2x15_Pitch2.54mm_SMD, F.Cu at (134.6, 105.4)
- added U1: AD9200JRSZ, Housings_SSOP:SSOP-28_5.3x10.2mm_Pitch0.65mm, B.Cu at (158.8, 105.4)
Other:
- board outline added: 125.7 x 94 mm
- rule pad_to_mask_clearance: 0.2 -> 0

Commit message: autoplaced
Routing:
- net /analog-ground: track 0.00 -> 137.3 mm, vias 0 -> 1
- net /upper-ref-V: track 0.00 -> 101.2 mm, vias 0 -> 1
- net /lower-ref-V: track 0.00 -> 74.9 mm, vias 0 -> 2
- net Net-(J1-Pad28): track 0.00 -> 55.4 mm, vias 0 -> 1
- net Net-(J1-Pad25): track 0.00 -> 45.1 mm, vias 0 -> 1
- net Net-(J1-Pad1): track 0.00 -> 42.7 mm, vias 0 -> 1
- net Net-(J1-Pad24): track 0.00 -> 39.5 mm, vias 0 -> 1
- net Net-(J1-Pad26): track 0.00 -> 38.5 mm, vias 0 -> 1
- net Net-(J1-Pad22): track 0.00 -> 37.7 mm, vias 0 -> 1
- net Net-(J1-Pad19): track 0.00 -> 37.4 mm, vias 0 -> 1
- net Net-(J1-Pad27): track 0.00 -> 36.8 mm, vias 0 -> 1
- net Net-(J1-Pad3): track 0.00 -> 36.7 mm, vias 0 -> 1
- net Net-(J1-Pad23): track 0.00 -> 35.3 mm, vias 0 -> 1
- net Net-(J1-Pad18): track 0.00 -> 34.1 mm, vias 0 -> 1
- net Net-(J1-Pad12): track 0.00 -> 33.5 mm, vias 0 -> 1
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Other:
- board size 125.7 x 94 mm -> 73.7 x 57.2 mm
