File: KIKAD-pcb/sampler.sch (KiCad schematic (older format))
At the start: 7 parts, among them J1 CONN_02X15, U1 AD9200JRSZ

Commit message: next attempt with eagle
Parts:
- C1, C2, C3, C4: footprint Capacitors_THT:C_Rect_L10.0mm_W2.5mm_P7.50mm_MKS4 -> Capacitors_SMD:C_0805
- C5: footprint Capacitors_THT:C_Rect_L26.5mm_W8.5mm_P22.50mm_MKS4 -> Capacitors_SMD:C_0603
- J1: footprint Socket_Strips:Socket_Strip_Straight_2x15_Pitch2.54mm_SMD -> Pin_Headers:Pin_Header_Straight_2x15_Pitch2.54mm_SMD
Changed lines of the file:
@@
 LIBS:contrib
 LIBS:valves
+LIBS:sampler-cache
 EELAYER 25 0
 EELAYER END
@@
 F 0 "J1" H 2300 3250 50  0000 C CNN
 F 1 "CONN_02X15" V 2300 2450 50  0000 C CNN
-F 2 "Socket_Strips:Socket_Strip_Straight_2x15_Pitch2.54mm_SMD" H 2300 1300 50  0001 C CNN
+F 2 "Pin_Headers:Pin_Header_Straight_2x15_Pitch2.54mm_SMD" H 2300 1300 50  0001 C CNN
 F 3 "" H 2300 1300 50  0001 C CNN
 	1    2300 2450
@@
 F 0 "C1" H 10275 1800 50  0000 L CNN
 F 1 "0.1uF" H 10275 1600 50  0000 L CNN
-F 2 "Capacitors_THT:C_Rect_L10.0mm_W2.5mm_P7.50mm_MKS4" H 10288 1550 50  0001 C CNN
+F 2 "Capacitors_SMD:C_0805" H 10288 1550 50  0001 C CNN
 F 3 "" H 10250 1700 50  0001 C CNN
 	1    10250 1700
@@
 F 0 "C2" H 10025 2500 50  0000 L CNN
 F 1 "0.1uF" H 10025 2300 50  0000 L CNN
-F 2 "Capacitors_THT:C_Rect_L10.0mm_W2.5mm_P7.50mm_MKS4" H 10038 2250 50  0001 C CNN
+F 2 "Capacitors_SMD:C_0805" H 10038 2250 50  0001 C CNN
 F 3 "" H 10000 2400 50  0001 C CNN
 	1    10000 2400
@@
 F 0 "C3" H 10025 3150 50  0000 L CNN
 F 1 "0.1uF" H 10025 2950 50  0000 L CNN
-F 2 "Capacitors_THT:C_Rect_L10.0mm_W2.5mm_P7.50mm_MKS4" H 10038 2900 50  0001 C CNN
+F 2 "Capacitors_SMD:C_0805" H 10038 2900 50  0001 C CNN
 F 3 "" H 10000 3050 50  0001 C CNN
 	1    10000 3050
@@
 F 0 "C5" H 10375 3150 50  0000 L CNN
 F 1 "10uF" H 10375 2950 50  0000 L CNN
-F 2 "Capacitors_THT:C_Rect_L26.5mm_W8.5mm_P22.50mm_MKS4" H 10388 2900 50  0001 C CNN
+F 2 "Capacitors_SMD:C_0603" H 10388 2900 50  0001 C CNN
 F 3 "" H 10350 3050 50  0001 C CNN
 	1    10350 3050
@@
 F 0 "C4" H 10025 3850 50  0000 L CNN
 F 1 "0.1uF" H 10025 3650 50  0000 L CNN
-F 2 "Capacitors_THT:C_Rect_L10.0mm_W2.5mm_P7.50mm_MKS4" H 10038 3600 50  0001 C CNN
+F 2 "Capacitors_SMD:C_0805" H 10038 3600 50  0001 C CNN
 F 3 "" H 10000 3750 50  0001 C CNN
 	1    10000 3750
